File: atlas.kicad_sch (KiCad schematic)
At the start: 230 parts

Commit message: First try for change from HasanDogruel
Parts:
- gave numbers to parts that had none: 1
Changed lines of the file:
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@@
   (symbol (lib_id "robot-eagle-import:JP1EJP1_SHORT") (at 344.17 245.11 0) (unit 1)
     (in_bom yes) (on_board yes)
-    (property "Reference" "JP?" (id 0) (at 342.9 245.11 90)
+    (property "Reference" "JP2" (id 0) (at 342.9 245.11 90)
       (effects (font (size 1.778 1.5113)) (justify left bottom))
     )
@@
       (reference "J?") (unit 1) (value "PINHD-1X10") (footprint "robot:1X10")
     )
-    (path "/2ef0e727-eb6c-4324-a6ba-f30c0bb34322"
-      (reference "JP?") (unit 1) (value "SHORT") (footprint "robot:JP1_SHORT")
-    )
     (path "/498bd9bb-ff7e-45f5-92c1-b16ac6c3913f"
+      (reference "JP2") (unit 1) (value "SHORT") (footprint "robot:JP1_SHORT")
+    )
+    (path "/2ef0e727-eb6c-4324-a6ba-f30c0bb34322"
       (reference "JP?") (unit 1) (value "SHORT") (footprint "robot:JP1_SHORT")
     )

Commit message: Jack Names Update
Parts:
- gave numbers to parts that had none: 98
Connections:
- net GIOA_3/N2HET2_2: no longer RP11.4 (2)
- net MDIO: no longer RP11.8 (2)
- net MII_CRS: no longer RP11.12 (2)
- net MII_RX_DV: no longer RP11.10 (2)
- net MII_RX_ER: no longer RP11.14 (2)
- net MII_TXD_2: now also U4.6 (TXD_3); no longer U4.5 (TXD_2)
- net MII_TXD_3: now also U4.5 (TXD_2); no longer U4.6 (TXD_3)
Other:
- note added: "DNP"
- note added: "GND"
- moved on the sheet: R7
